File: electronics/polythene_sensor/polythene_sensor.sch (KiCad schematic (older format))
At the start: 7 parts, among them J1 Conn_02x16_Counter_Clockwise

Commit message: Board ready
Signed-off-by: byteofsoren <r00tr4t@gmail.com>
Parts:
- added Raref1: 10k, Potentiometer_THT:Potentiometer_Piher_PT-15-V02_Vertical, symbol Device:R_POT_TRIM
- Jfpow1: footprint polythene_sensor:Cage_clamp_2pole -> polythene_sensor:MOLEX_104188
Connections:
- net +5V: now also Raref1.1
- net GND: now also Raref1.3; no longer A1.2 (IOREF), A1.30 (AREF)
- new net: A1.30 (AREF), Raref1.2
- no-connect marks 15 -> 16
Changed lines of the file:
@@
 EESchema Schematic File Version 4
+LIBS:polythene_sensor-cache
 EELAYER 29 0
 EELAYER END
@@
 Comment4 ""
 $EndDescr
-$Comp
-L power:GND #PWR03
-U 1 1 5CCDFED3
-P 3100 4800
-F 0 "#PWR03" H 3100 4550 50  0001 C CNN
-F 1 "GND" H 3105 4627 50  0000 C CNN
-F 2 "" H 3100 4800 50  0001 C CNN
-F 3 "" H 3100 4800 50  0001 C CNN
-	1    3100 4800
-	-1   0    0    -1
-$EndComp
-$Comp
-L power:GND #PWR05
-U 1 1 5CCE096E
-P 5950 2600
-F 0 "#PWR05" H 5950 2350 50  0001 C CNN
-F 1 "GND" H 5955 2427 50  0000 C CNN
-F 2 "" H 5950 2600 50  0001 C CNN
-F 3 "" H 5950 2600 50  0001 C CNN
-	1    5950 2600
-	1    0    0    1
-$EndComp
 Wire Wire Line
 	8650 3000 9150 3000
@@
 	6550 4600 6550 4700
 Wire Wire Line
-	6550 4700 7000 4700
-Wire Wire Line
 	7150 4700 7150 4600
 Wire Wire Line
@@
 L power:GND #PWR07
 U 1 1 5CDC317B
-P 7000 4700
-F 0 "#PWR07" H 7000 4450 50  0001 C CNN
-F 1 "GND" H 7005 4527 50  0000 C CNN
-F 2 "" H 7000 4700 50  0001 C CNN
-F 3 "" H 7000 4700 50  0001 C CNN
-	1    7000 4700
-	1    0    0    -1
-$EndComp
-Connection ~ 7000 4700
-Wire Wire Line
-	7000 4700 7150 4700
-$Comp
-L Connector_Generic:Conn_01x02 Jfpow1
-U 1 1 5CDDD1C6
-P 2100 3200
-F 0 "Jfpow1" H 2018 3417 50  0000 C CNN
-F 1 "Conn_01x02" H 2018 3326 50  0000 C CNN
-F 2 "polythene_sensor:Cage_clamp_2pole" H 2100 3200 50  0001 C CNN
-F 3 "https://www.elfa.se/Web/Downloads/_t/ds/2061-601_998-404_eng_tds.pdf" H 2100 3200 50  0001 C CNN
-	1    2100 3200
-	-1   0    0    -1
-$EndComp
-$Comp
-L power:GND #PWR01
-U 1 1 5CDDE928
-P 2300 3300
-F 0 "#PWR01" H 2300 3050 50  0001 C CNN
-F 1 "GND" H 2305 3127 50  0000 C CNN
-F 2 "" H 2300 3300 50  0001 C CNN
-F 3 "" H 2300 3300 50  0001 C CNN
-	1    2300 3300
-	-1   0    0    -1
-$EndComp
-Wire Wire Line
-	2300 3200 2600 3200
-$Comp
-L northspawn_v2-cache:power_+5V #PWR08
-U 1 1 5CDF49A1
-P 7950 2150
-F 0 "#PWR08" H 7950 2000 50  0001 C CNN
-F 1 "power_+5V" H 7965 2323 50  0000 C CNN
-F 2 "" H 7950 2150 50  0001 C CNN
-F 3 "" H 7950 2150 50  0001 C CNN
-	1    7950 2150
-	1    0    0    -1
-$EndComp
-$Comp
-L northspawn_v2-cache:power_+5V #PWR02
-U 1 1 5CDF5A3E
-P 3100 2450
-F 0 "#PWR02" H 3100 2300 50  0001 C CNN
-F 1 "power_+5V" H 3115 2623 50  0000 C CNN
-F 2 "" H 3100 2450 50  0001 C CNN
-F 3 "" H 3100 2450 50  0001 C CNN
-	1    3100 2450
-	1    0    0    -1
-$EndComp
-$Comp
-L northspawn_v2-cache:power_+5V #PWR04
-U 1 1 5CDF7B84
-P 5250 4800
-F 0 "#PWR04" H 5250 4650 50  0001 C CNN
-F 1 "power_+5V" H 5265 4973 50  0000 C CNN
-F 2 "" H 5250 4800 50  0001 C CNN
-F 3 "" H 5250 4800 50  0001 C CNN
-	1    5250 4800
-	1    0    0    -1
-$EndComp
-Wire Wire Line
-	5950 4950 5250 4950
-Wire Wire Line
-	5250 4950 5250 4800
-Wire Wire Line
-	3100 2450 3100 2700
-Wire Wire Line
-	7950 2150 7950 2400
-$Comp
-L power:GND #PWR06
-U 1 1 5CE03B42
-P 7000 3300
-F 0 "#PWR06" H 7000 3050 50  0001 C CNN
-F 1 "GND" H 7005 3127 50  0000 C CNN
-F 2 "" H 7000 3300 50  0001 C CNN
-F 3 "" H 7000 3300 50  0001 C CNN
-	1    7000 3300
-	1    0    0    -1
-$EndComp
-Wire Wire Line
-	7650 3200 7500 3200
-Wire Wire Line
-	7000 3200 7000 3300
+P 7000 4800
+F 0 "#PWR07" H 7000 4550 50  0001 C CNN
+F 1 "GND" H 7005 4627 50  0000 C CNN
+F 2 "" H 7000 4800 50  0001 C CNN
+F 3 "" H 7000 4800 50  0001 C CNN
+	1    7000 4800
+	1    0    0    -1
+$EndComp
 Wire Wire Line
 	4800 4500 5450 4500
@@
 Wire Wire Line
 	4800 3900 5450 3900
-Wire Wire Line
-	5950 4800 5950 4950
 Wire Wire Line
 	4800 3700 5450 3700
@@
 	-1   0    0    1
 $EndComp
-Wire Wire Line
-	7650 3000 7500 3000
-Wire Wire Line
-	7500 3000 7500 3200
-Connection ~ 7500 3200
-Wire Wire Line
-	7500 3200 7000 3200
 NoConn ~ 8650 2800
 NoConn ~ 8650 2900
@@
 Wire Wire Line
 	8250 4500 8250 4600
-Wire Wire Line
-	8250 4600 8150 4600
-Wire Wire Line
-	8150 4600 8050 4600
-Connection ~ 8150 4600
-Wire Wire Line
-	8150 4500 8150 4600
 Connection ~ 8050 4600
 $Comp
@@
 	-1   0    0    -1
 $EndComp
-Wire Bus Line
-	2200 3700 2200 5200
-Wire Bus Line
-	6800 3200 6800 5200
-Wire Bus Line
-	9250 3100 9250 5200
 $Comp
 L Connector_Generic:Conn_02x16_Counter_Clockwise J1
@@
 	1    0    0    -1
 $EndComp
+NoConn ~ 7650 3000
+$Comp
+L Connector_Generic:Conn_01x02 Jfpow1
+U 1 1 5CD4E46C
+P 1950 3200
+F 0 "Jfpow1" H 1868 3417 50  0000 C CNN
+F 1 "Conn_01x02" H 1868 3326 50  0000 C CNN
+F 2 "polythene_sensor:MOLEX_104188" H 1950 3200 50  0001 C CNN
+F 3 "~" H 1950 3200 50  0001 C CNN
+	1    1950 3200
+	-1   0    0    -1
+$EndComp
+Wire Wire Line
+	2150 3200 2600 3200
+$Comp
+L Device:R_POT_TRIM Raref1
+U 1 1 5CD68CF7
+P 7100 2500
+F 0 "Raref1" H 7031 2546 50  0000 R CNN
+F 1 "10k" H 7031 2455 50  0000 R CNN
+F 2 "Potentiometer_THT:Potentiometer_Piher_PT-15-V02_Vertical" H 7100 2500 50  0001 C CNN
+F 3 "~" H 7100 2500 50  0001 C CNN
+	1    7100 2500
+	1    0    0    -1
+$EndComp
+Wire Wire Line
+	7350 2500 7350 3200
+Wire Wire Line
+	7350 3200 7650 3200
+Wire Wire Line
+	7250 2500 7350 2500
+$Comp
+L power:GND #PWR0104
+U 1 1 5CD80D9F
+P 5950 2600
+F 0 "#PWR0104" H 5950 2350 50  0001 C CNN
+F 1 "GND" H 5955 2427 50  0000 C CNN
+F 2 "" H 5950 2600 50  0001 C CNN
+F 3 "" H 5950 2600 50  0001 C CNN
+	1    5950 2600
+	-1   0    0    1
+$EndComp
+Wire Wire Line
+	8050 4600 8150 4600
+Wire Wire Line
+	8150 4500 8150 4600
+Connection ~ 8150 4600
+Wire Wire Line
+	8150 4600 8250 4600
+$Comp
+L power:GND #PWR0107
+U 1 1 5CDA49EE
+P 3800 5000
+F 0 "#PWR0107" H 3800 4750 50  0001 C CNN
+F 1 "GND" H 3805 4827 50  0000 C CNN
+F 2 "" H 3800 5000 50  0001 C CNN
+F 3 "" H 3800 5000 50  0001 C CNN
+	1    3800 5000
+	1    0    0    -1
+$EndComp
+Wire Wire Line
+	6550 4700 7000 4700
+Wire Wire Line
+	7000 4800 7000 4700
+Connection ~ 7000 4700
+Wire Wire Line
+	7000 4700 7150 4700
+$Comp
+L power:GND #PWR0108
+U 1 1 5CDBFF1F
+P 2400 3350
+F 0 "#PWR0108" H 2400 3100 50  0001 C CNN
+F 1 "GND" H 2405 3177 50  0000 C CNN
+F 2 "" H 2400 3350 50  0001 C CNN
+F 3 "" H 2400 3350 50  0001 C CNN
+	1    2400 3350
+	1    0    0    -1
+$EndComp
+Wire Wire Line
+	3100 4800 3100 4900
+Wire Wire Line
+	3100 4900 3800 4900
+Wire Wire Line
+	3800 4900 3800 5000
+Wire Wire Line
+	2150 3300 2400 3300
+Wire Wire Line
+	2400 3300 2400 3350
+$Comp
+L power:GND #PWR0101
+U 1 1 5CD749E8
+P 7100 2650
+F 0 "#PWR0101" H 7100 2400 50  0001 C CNN
+F 1 "GND" H 7105 2477 50  0000 C CNN
+F 2 "" H 7100 2650 50  0001 C CNN
+F 3 "" H 7100 2650 50  0001 C CNN
+	1    7100 2650
+	-1   0    0    -1
+$EndComp
+$Comp
+L power:+5V #PWR0102
+U 1 1 5CE6FAF2
+P 7950 2100
+F 0 "#PWR0102" H 7950 1950 50  0001 C CNN
+F 1 "+5V" H 7965 2273 50  0000 C CNN
+F 2 "" H 7950 2100 50  0001 C CNN
+F 3 "" H 7950 2100 50  0001 C CNN
+	1    7950 2100
+	1    0    0    -1
+$EndComp
+Wire Wire Line
+	7950 2400 7950 2100
+$Comp
+L power:+5V #PWR0103
+U 1 1 5CE74282
+P 7100 2100
+F 0 "#PWR0103" H 7100 1950 50  0001 C CNN
+F 1 "+5V" H 7115 2273 50  0000 C CNN
+F 2 "" H 7100 2100 50  0001 C CNN
+F 3 "" H 7100 2100 50  0001 C CNN
+	1    7100 2100
+	1    0    0    -1
+$EndComp
+Wire Wire Line
+	7100 2100 7100 2350
+$Comp
+L power:PWR_FLAG #FLG01
+U 1 1 5CE879D2
+P 8400 4600
+F 0 "#FLG01" H 8400 4675 50  0001 C CNN
+F 1 "PWR_FLAG" V 8400 4728 50  0000 L CNN
+F 2 "" H 8400 4600 50  0001 C CNN
+F 3 "~" H 8400 4600 50  0001 C CNN
+	1    8400 4600
+	0    1    1    0
+$EndComp
+Wire Wire Line
+	8400 4600 8250 4600
+Connection ~ 8250 4600
+$Comp
+L power:+5V #PWR01
+U 1 1 5CE919FA
+P 5650 4950
+F 0 "#PWR01" H 5650 4800 50  0001 C CNN
+F 1 "+5V" H 5665 5123 50  0000 C CNN
+F 2 "" H 5650 4950 50  0001 C CNN
+F 3 "" H 5650 4950 50  0001 C CNN
+	1    5650 4950
+	1    0    0    -1
+$EndComp
+Wire Wire Line
+	5650 4950 5650 5050
+Wire Wire Line
+	5650 5050 5950 5050
+Wire Wire Line
+	5950 5050 5950 4800
+$Comp
+L power:+5V #PWR02
+U 1 1 5CE9BBAC
+P 3100 2550
+F 0 "#PWR02" H 3100 2400 50  0001 C CNN
+F 1 "+5V" H 3115 2723 50  0000 C CNN
+F 2 "" H 3100 2550 50  0001 C CNN
+F 3 "" H 3100 2550 50  0001 C CNN
+	1    3100 2550
+	1    0    0    -1
+$EndComp
+Wire Wire Line
+	3100 2550 3100 2700
+Wire Bus Line
+	2200 3700 2200 5200
+Wire Bus Line
+	6800 3200 6800 5200
+Wire Bus Line
+	9250 3100 9250 5200
 $EndSCHEMATC

Commit message: Updated parts
Signed-off-by: byteofsoren <r00tr4t@gmail.com>
Parts:
- removed A1: Arduino_UNO_R3, Module:Arduino_UNO_R3, symbol MCU_Module:Arduino_UNO_R3
- removed J1: Conn_02x16_Counter_Clockwise, One27:One27_male_32pin, symbol Connector_Generic:Conn_02x16_Counter_Clockwise
- removed Raref1: 10k, Potentiometer_THT:Potentiometer_Piher_PT-15-V02_Vertical, symbol Device:R_POT_TRIM
- added J?: Conn_02x18_Odd_Even, Connector_PinHeader_2.54mm:PinHeader_2x18_P2.54mm_Vertical_SMD, symbol Connector_Generic:Conn_02x18_Odd_Even
- added J?: Conn_02x08_Odd_Even, symbol Connector_Generic:Conn_02x08_Odd_Even
Connections:
- net +5V: now also J?.1 (Pin_1), J?.16 (Pin_16)
- net EN: now also J?.12 (Pin_12), J?.5 (Pin_5)
- net GND: now also J?.15 (Pin_15), J?.2 (Pin_2)
- net S0: now also J?.13 (Pin_13)
- net S1: now also J?.11 (Pin_11)
- net S2: now also J?.9 (Pin_9)
- net S3: now also J?.7 (Pin_7)
- net S4: now also J?.10 (Pin_10)
- net S5: now also J?.8 (Pin_8)
- net S6: now also J?.6 (Pin_6)
- net S7: now also J?.4 (Pin_4)
- net at Uin1.16 (I15): now also J?.33 (Pin_33)
- net at Uin1.17 (I14): now also J?.31 (Pin_31)
- net at Uin1.18 (I13): now also J?.29 (Pin_29)
- net at Uin1.19 (I12): now also J?.27 (Pin_27)
- net at Uin1.2 (I7): now also J?.17 (Pin_17)
- net at Uin1.20 (I11): now also J?.25 (Pin_25)
- net at Uin1.21 (I10): now also J?.23 (Pin_23)
- net at Uin1.22 (I9): now also J?.21 (Pin_21)
- net at Uin1.23 (I8): now also J?.19 (Pin_19)
- net at Uin1.3 (I6): now also J?.15 (Pin_15)
- net at Uin1.4 (I5): now also J?.13 (Pin_13)
- net at Uin1.5 (I4): now also J?.11 (Pin_11)
- net at Uin1.6 (I3): now also J?.9 (Pin_9)
- net at Uin1.7 (I2): now also J?.7 (Pin_7)
- net at Uin1.8 (I1): now also J?.5 (Pin_5)
- net at Uin1.9 (I0): now also J?.3 (Pin_3)
- net at Dprot1.1 (K), Rref1.1, Uout1.1 (COM): now also J?.14 (Pin_14), J?.3 (Pin_3)
- net at Uout1.16 (I15): now also J?.4 (Pin_4)
- net at Uout1.17 (I14): now also J?.6 (Pin_6)
- net at Uout1.18 (I13): now also J?.8 (Pin_8)
- net at Uout1.19 (I12): now also J?.10 (Pin_10)
- net at Uout1.2 (I7): now also J?.20 (Pin_20)
- net at Uout1.20 (I11): now also J?.12 (Pin_12)
- net at Uout1.21 (I10): now also J?.14 (Pin_14)
- net at Uout1.22 (I9): now also J?.16 (Pin_16)
- net at Uout1.23 (I8): now also J?.18 (Pin_18)
- net at Uout1.3 (I6): now also J?.22 (Pin_22)
- net at Uout1.4 (I5): now also J?.24 (Pin_24)
- net at Uout1.5 (I4): now also J?.26 (Pin_26)
- net at Uout1.6 (I3): now also J?.28 (Pin_28)
- net at Uout1.7 (I2): now also J?.30 (Pin_30)
- net at Uout1.8 (I1): now also J?.32 (Pin_32)
- net at Uout1.9 (I0): now also J?.34 (Pin_34)
- no-connect marks 16 -> 0
Other:
- note added: "12 May 2019"
- note added: "MUX to arduino connection sheame."
- note added: "Polythene sensor sheald for Arduino"

Commit message: Updated in the electronics
Signed-off-by: byteofsoren <r00tr4t@gmail.com>
Parts:
- gave numbers to parts that had none: 2
Connections:
- no-connect marks 0 -> 4
Changed lines of the file:
@@
 	6800 5200 7800 5200
 $Comp
-L Connector_Generic:Conn_02x18_Odd_Even J?
+L Connector_Generic:Conn_02x18_Odd_Even J1
 U 1 1 5CEEFA8E
 P 4500 3700
-F 0 "J?" H 4550 4717 50  0000 C CNN
+F 0 "J1" H 4550 4717 50  0000 C CNN
 F 1 "Conn_02x18_Odd_Even" H 4550 4626 50  0000 C CNN
 F 2 "Connector_PinHeader_2.54mm:PinHeader_2x18_P2.54mm_Vertical_SMD" H 4500 3700 50  0001 C CNN
@@
 $EndComp
 $Comp
-L Connector_Generic:Conn_02x08_Odd_Even J?
+L Connector_Generic:Conn_02x08_Odd_Even J2
 U 1 1 5CF151F3
 P 8850 3850
-F 0 "J?" H 8900 4367 50  0000 C CNN
+F 0 "J2" H 8900 4367 50  0000 C CNN
 F 1 "Conn_02x08_Odd_Even" H 8900 4276 50  0000 C CNN
 F 2 "" H 8850 3850 50  0001 C CNN
@@
 $EndComp
 $Comp
-L power:GND #PWR?
+L power:GND #PWR04
 U 1 1 5CF15D69
 P 8500 4450
-F 0 "#PWR?" H 8500 4200 50  0001 C CNN
+F 0 "#PWR04" H 8500 4200 50  0001 C CNN
 F 1 "GND" H 8505 4277 50  0000 C CNN
 F 2 "" H 8500 4450 50  0001 C CNN
@@
 $EndComp
 $Comp
-L power:+5V #PWR?
+L power:+5V #PWR03
 U 1 1 5CF16B03
 P 8250 3350
-F 0 "#PWR?" H 8250 3200 50  0001 C CNN
+F 0 "#PWR03" H 8250 3200 50  0001 C CNN
 F 1 "+5V" H 8265 3523 50  0000 C CNN
 F 2 "" H 8250 3350 50  0001 C CNN
@@
 $EndComp
 $Comp
-L power:+5V #PWR?
+L power:+5V #PWR05
 U 1 1 5CF172C7
 P 9400 3350
-F 0 "#PWR?" H 9400 3200 50  0001 C CNN
+F 0 "#PWR05" H 9400 3200 50  0001 C CNN
 F 1 "+5V" H 9415 3523 50  0000 C CNN
 F 2 "" H 9400 3350 50  0001 C CNN
@@
 $EndComp
 $Comp
-L power:GND #PWR?
+L power:GND #PWR06
 U 1 1 5CF179B3
 P 9650 4500
-F 0 "#PWR?" H 9650 4250 50  0001 C CNN
+F 0 "#PWR06" H 9650 4250 50  0001 C CNN
 F 1 "GND" H 9655 4327 50  0000 C CNN
 F 2 "" H 9650 4500 50  0001 C CNN
@@
 Wire Wire Line
 	9950 4050 9150 4050
-Wire Wire Line
-	9150 4150 10150 4150
-Wire Bus Line
-	2200 3700 2200 5200
-Wire Bus Line
-	6800 3200 6800 5200
-Wire Bus Line
-	10050 3700 10050 5200
-Wire Bus Line
-	7800 3700 7800 5200
 Text Label 8350 4150 0    50   ~ 0
 S0
@@
 Text Label 9200 4050 0    50   ~ 0
 EN
+NoConn ~ 4300 2900
+NoConn ~ 4800 2900
+NoConn ~ 4300 4600
+NoConn ~ 4800 4600
+Wire Wire Line
+	9150 4150 10150 4150
+Wire Bus Line
+	2200 3700 2200 5200
+Wire Bus Line
+	6800 3200 6800 5200
+Wire Bus Line
+	10050 3700 10050 5200
+Wire Bus Line
+	7800 3700 7800 5200
+$Comp
+L power:PWR_FLAG #FLG0101
+U 1 1 5CE2AD6B
+P 8250 3350
+F 0 "#FLG0101" H 8250 3425 50  0001 C CNN
+F 1 "PWR_FLAG" V 8150 3600 50  0000 L CNN
+F 2 "" H 8250 3350 50  0001 C CNN
+F 3 "~" H 8250 3350 50  0001 C CNN
+	1    8250 3350
+	0    1    1    0
+$EndComp
+Connection ~ 8250 3350
 $EndSCHEMATC
