File: electronics/polythene_sensor/polythene_sensor.kicad_pcb (KiCad board)
At the start: 2 copper layers, 7 parts, among them J1 Conn_02x16_Counter_Clockwise

Commit message: Board ready
Signed-off-by: byteofsoren <r00tr4t@gmail.com>
Parts:
- added Raref1: 10k, Potentiometer_THT:Potentiometer_Piher_PT-15-V02_Vertical, F.Cu at (121.2, 80.3)
- Jfpow1: footprint polythene_sensor:Cage_clamp_2pole -> polythene_sensor:MOLEX_104188
- moved Jfpow1 12.2 mm to (135.8, 111.4), turned to 270 degrees
Connections:
- A1 pad 2: GND -> Net-(A1-Pad2)
- A1 pad 30: GND -> Net-(A1-Pad30)
Routing:
- net +5V: track 81.3 -> 147.5 mm
- net Net-(Jfpow1-Pad1): track 53.7 -> 37.0 mm, vias 4 -> 2
- net Net-(A1-Pad30): track 0.00 -> 12.3 mm
- net GND: track 174.8 -> 166.1 mm
- net /S3: track 50.4 -> 52.2 mm
- net /S6: track 58.0 -> 56.6 mm
- net /S7: track 54.3 -> 53.1 mm

Commit message: Updated parts
Signed-off-by: byteofsoren <r00tr4t@gmail.com>
Parts:
- moved Rref1 15.9 mm to (179.5, 110.9), turned to 90 degrees
- moved Dprot1 10.8 mm to (173.8, 110.7), turned to 90 degrees
Routing:
- net Net-(A1-Pad9): track 29.9 -> 57.9 mm
- net GND: track 166.1 -> 184.5 mm
Other:
- board text removed: "FoamSens"
Changed lines of the file:
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@@
   (general
     (thickness 1.6)
-    (drawings 1)
-    (tracks 405)
+    (drawings 0)
+    (tracks 413)
     (zones 0)
     (modules 8)
@@
   )
   (module Diodes_SMD:D_SOD-123 (layer F.Cu)
-    (at 163.6522 114.3127 180)
+    (at 173.82744 110.7196 90)
     (descr SOD-123)
     (tags SOD-123)
     (attr smd)
-    (fp_text reference Dprot1 (at 0 -2) (layer F.SilkS)
-      (effects (font (size 1 1) (thickness 0.15)))
-    )
-    (fp_text value BZT52Bxx (at 0 2.1) (layer F.Fab)
-      (effects (font (size 1 1) (thickness 0.15)))
-    )
-    (fp_text user %R (at 0 -2) (layer F.Fab)
+    (fp_text reference Dprot1 (at 0 -2 90) (layer F.SilkS)
+      (effects (font (size 1 1) (thickness 0.15)))
+    )
+    (fp_text value BZT52Bxx (at 0 2.1 90) (layer F.Fab)
+      (effects (font (size 1 1) (thickness 0.15)))
+    )
+    (fp_text user %R (at 0 -2 90) (layer F.Fab)
       (effects (font (size 1 1) (thickness 0.15)))
     )
@@
     (fp_line (start -2.25 1) (end 1.65 1) (layer F.SilkS) (width 0.12))
     (fp_line (start -2.25 -1) (end 1.65 -1) (layer F.SilkS) (width 0.12))
-    (pad 1 smd rect (at -1.65 0 180) (size 0.9 1.2) (layers F.Cu F.Paste F.Mask)
+    (pad 1 smd rect (at -1.65 0 90) (size 0.9 1.2) (layers F.Cu F.Paste F.Mask)
       (net 3 "Net-(A1-Pad9)"))
-    (pad 2 smd rect (at 1.65 0 180) (size 0.9 1.2) (layers F.Cu F.Paste F.Mask)
+    (pad 2 smd rect (at 1.65 0 90) (size 0.9 1.2) (layers F.Cu F.Paste F.Mask)
       (net 2 GND))
     (model ${KISYS3DMOD}/Diodes_SMD.3dshapes/D_SOD-123.wrl
@@
   )
   (module Resistors_SMD:R_0805_HandSoldering (layer F.Cu)
-    (at 163.5633 110.5662 180)
+    (at 179.47132 110.87736 90)
     (descr "Resistor SMD 0805, hand soldering")
     (tags "resistor 0805")
     (attr smd)
-    (fp_text reference Rref1 (at 0 -1.7) (layer F.SilkS)
-      (effects (font (size 1 1) (thickness 0.15)))
-    )
-    (fp_text value R (at 0 1.75) (layer F.Fab)
+    (fp_text reference Rref1 (at 0 -1.7 90) (layer F.SilkS)
+      (effects (font (size 1 1) (thickness 0.15)))
+    )
+    (fp_text value R (at 0 1.75 90) (layer F.Fab)
       (effects (font (size 1 1) (thickness 0.15)))
     )
@@
     (fp_line (start 1 0.62) (end -1 0.62) (layer F.Fab) (width 0.1))
     (fp_line (start -1 0.62) (end -1 -0.62) (layer F.Fab) (width 0.1))
-    (fp_text user %R (at 0 0) (layer F.Fab)
+    (fp_text user %R (at 0 0 90) (layer F.Fab)
       (effects (font (size 0.5 0.5) (thickness 0.075)))
     )
-    (pad 2 smd rect (at 1.35 0 180) (size 1.5 1.3) (layers F.Cu F.Paste F.Mask)
-      (net 2 GND))
-    (pad 1 smd rect (at -1.35 0 180) (size 1.5 1.3) (layers F.Cu F.Paste F.Mask)
+    (pad 2 smd rect (at 1.35 0 90) (size 1.5 1.3) (layers F.Cu F.Paste F.Mask)
+      (net 2 GND))
+    (pad 1 smd rect (at -1.35 0 90) (size 1.5 1.3) (layers F.Cu F.Paste F.Mask)
       (net 3 "Net-(A1-Pad9)"))
     (model ${KISYS3DMOD}/Resistors_SMD.3dshapes/R_0805.wrl
@@
       (net 2 GND))
   )
-  (gr_text FoamSens (at 177.2158 111.7092) (layer F.Cu)
-    (effects (font (size 1.5 1.5) (thickness 0.3)))
-  )
   (via (at 156.7815 105.8672) (size 2) (drill 1.8) (layers F.Cu B.Cu) (net 0))
   (via (at 156.7688 83.1215) (size 2) (drill 1.8) (layers F.Cu B.Cu) (net 0))
@@
   (via (at 163.3093 107.5944) (size 1.5) (drill 1) (layers F.Cu B.Cu) (net 2))
   (segment (start 163.3093 95.828385) (end 163.3093 107.5944) (width 0.6) (layer B.Cu) (net 2))
-  (segment (start 162.2133 108.6904) (end 162.2133 110.5662) (width 0.6) (layer F.Cu) (net 2))
-  (segment (start 163.3093 107.5944) (end 162.2133 108.6904) (width 0.6) (layer F.Cu) (net 2))
-  (segment (start 162.2133 114.1016) (end 162.0022 114.3127) (width 0.6) (layer F.Cu) (net 2))
-  (segment (start 162.2133 110.5662) (end 162.2133 114.1016) (width 0.6) (layer F.Cu) (net 2))
-  (segment (start 162.0022 117.6792) (end 162.0139 117.6909) (width 0.6) (layer F.Cu) (net 2))
-  (segment (start 162.0022 114.3127) (end 162.0022 117.6792) (width 0.6) (layer F.Cu) (net 2))
-  (segment (start 162.0022 114.3127) (end 159.9311 114.3127) (width 0.6) (layer F.Cu) (net 2))
-  (segment (start 159.4739 114.7699) (end 159.4739 117.6909) (width 0.6) (layer F.Cu) (net 2))
   (segment (start 130.3465 89.838) (end 130.0607 90.1238) (width 0.6) (layer F.Cu) (net 2))
   (segment (start 130.7465 89.838) (end 130.3465 89.838) (width 0.6) (layer F.Cu) (net 2))
@@
   (segment (start 144.853481 111.195279) (end 156.397119 111.195279) (width 0.6) (layer F.Cu) (net 2))
   (segment (start 142.66468 113.38408) (end 144.853481 111.195279) (width 0.6) (layer F.Cu) (net 2))
-  (segment (start 156.397119 111.195279) (end 159.72282 114.52098) (width 0.6) (layer F.Cu) (net 2))
   (segment (start 140.31468 113.38408) (end 142.66468 113.38408) (width 0.6) (layer F.Cu) (net 2))
-  (segment (start 159.9311 114.3127) (end 159.72282 114.52098) (width 0.6) (layer F.Cu) (net 2))
-  (segment (start 159.72282 114.52098) (end 159.4739 114.7699) (width 0.6) (layer F.Cu) (net 2))
   (segment (start 124.292883 70.33004) (end 127.67056 73.707717) (width 0.6) (layer F.Cu) (net 2))
   (segment (start 121.22404 70.33004) (end 124.292883 70.33004) (width 0.6) (layer F.Cu) (net 2))
@@
   (segment (start 138.320839 76.238041) (end 132.59562 81.96326) (width 0.6) (layer F.Cu) (net 2))
   (segment (start 132.59562 81.96326) (end 124.79528 89.7636) (width 0.6) (layer F.Cu) (net 2))
-  (segment (start 164.9133 109.3162) (end 164.9476 109.2819) (width 0.6) (layer F.Cu) (net 3))
-  (segment (start 164.9133 110.5662) (end 164.9133 109.3162) (width 0.6) (layer F.Cu) (net 3))
-  (segment (start 164.9476 109.2819) (end 164.9476 107.6198) (width 0.6) (layer F.Cu) (net 3))
+  (segment (start 174.2852 109.52736) (end 173.82744 109.0696) (width 0.6) (layer F.Cu) (net 2))
+  (segment (start 179.47132 109.52736) (end 174.2852 109.52736) (width 0.6) (layer F.Cu) (net 2))
+  (segment (start 159.4739 114.27206) (end 156.397119 111.195279) (width 0.6) (layer F.Cu) (net 2))
+  (segment (start 159.4739 117.6909) (end 159.4739 114.27206) (width 0.6) (layer F.Cu) (net 2))
+  (segment (start 172.62744 109.0696) (end 172.4872 109.20984) (width 0.6) (layer F.Cu) (net 2))
+  (segment (start 173.82744 109.0696) (end 172.62744 109.0696) (width 0.6) (layer F.Cu) (net 2))
+  (segment (start 158.382558 109.20984) (end 156.397119 111.195279) (width 0.6) (layer F.Cu) (net 2))
+  (segment (start 172.4872 109.20984) (end 163.20516 109.20984) (width 0.6) (layer F.Cu) (net 2))
+  (segment (start 163.20516 109.20984) (end 158.382558 109.20984) (width 0.6) (layer F.Cu) (net 2))
+  (segment (start 163.3093 109.1057) (end 163.20516 109.20984) (width 0.6) (layer F.Cu) (net 2))
+  (segment (start 163.3093 107.5944) (end 163.3093 109.1057) (width 0.6) (layer F.Cu) (net 2))
+  (segment (start 159.4739 114.27206) (end 161.77006 114.27206) (width 0.6) (layer F.Cu) (net 2))
+  (segment (start 162.0139 114.5159) (end 162.0139 117.6909) (width 0.6) (layer F.Cu) (net 2))
+  (segment (start 161.77006 114.27206) (end 162.0139 114.5159) (width 0.6) (layer F.Cu) (net 2))
   (via (at 164.9476 107.6198) (size 1.5) (drill 1) (layers F.Cu B.Cu) (net 3))
   (via (at 164.9476 107.6198) (size 1.5) (drill 1) (layers F.Cu B.Cu) (net 3))
@@
   (segment (start 164.9476 96.8756) (end 165.347599 96.475601) (width 0.6) (layer F.Cu) (net 3))
   (segment (start 165.347599 96.475601) (end 167.074901 96.475601) (width 0.6) (layer F.Cu) (net 3))
-  (segment (start 164.9133 113.9238) (end 165.3022 114.3127) (width 0.6) (layer F.Cu) (net 3))
-  (segment (start 164.9133 110.5662) (end 164.9133 113.9238) (width 0.6) (layer F.Cu) (net 3))
-  (segment (start 166.3522 114.3127) (end 166.3776 114.3381) (width 0.6) (layer F.Cu) (net 3))
-  (segment (start 165.3022 114.3127) (end 166.3522 114.3127) (width 0.6) (layer F.Cu) (net 3))
-  (segment (start 166.3776 114.3381) (end 168.7195 114.3381) (width 0.6) (layer F.Cu) (net 3))
-  (segment (start 169.6339 115.2525) (end 169.6339 117.6909) (width 0.6) (layer F.Cu) (net 3))
-  (segment (start 168.7195 114.3381) (end 169.6339 115.2525) (width 0.6) (layer F.Cu) (net 3))
+  (segment (start 169.6339 117.6909) (end 169.6339 114.59718) (width 0.6) (layer F.Cu) (net 3))
+  (segment (start 171.86148 112.3696) (end 173.82744 112.3696) (width 0.6) (layer F.Cu) (net 3))
+  (segment (start 169.6339 114.59718) (end 171.86148 112.3696) (width 0.6) (layer F.Cu) (net 3))
+  (segment (start 179.32908 112.3696) (end 179.47132 112.22736) (width 0.6) (layer F.Cu) (net 3))
+  (segment (start 173.82744 112.3696) (end 179.32908 112.3696) (width 0.6) (layer F.Cu) (net 3))
+  (segment (start 179.47132 112.22736) (end 182.45328 112.22736) (width 0.6) (layer F.Cu) (net 3))
+  (segment (start 182.45328 112.22736) (end 183.12892 111.55172) (width 0.6) (layer F.Cu) (net 3))
+  (segment (start 183.12892 110.884958) (end 183.1086 110.864638) (width 0.6) (layer F.Cu) (net 3))
+  (segment (start 183.12892 111.55172) (end 183.12892 110.884958) (width 0.6) (layer F.Cu) (net 3))
+  (segment (start 183.1086 110.864638) (end 183.1086 107.17784) (width 0.6) (layer F.Cu) (net 3))
+  (segment (start 183.1086 107.17784) (end 181.43728 105.50652) (width 0.6) (layer F.Cu) (net 3))
+  (segment (start 166.00826 107.6198) (end 164.9476 107.6198) (width 0.6) (layer F.Cu) (net 3))
+  (segment (start 171.178188 107.6198) (end 166.00826 107.6198) (width 0.6) (layer F.Cu) (net 3))
+  (segment (start 173.291468 105.50652) (end 171.178188 107.6198) (width 0.6) (layer F.Cu) (net 3))
+  (segment (start 181.43728 105.50652) (end 173.291468 105.50652) (width 0.6) (layer F.Cu) (net 3))
   (segment (start 177.7365 88.713) (end 177.7365 89.838) (width 0.6) (layer F.Cu) (net 4))
   (segment (start 163.620196 82.71292) (end 171.73642 82.71292) (width 0.6) (layer F.Cu) (net 4))

Commit message: Updated in the electronics
Signed-off-by: byteofsoren <r00tr4t@gmail.com>
Parts:
- removed A1: Arduino_UNO_R3, Module:Arduino_UNO_R3
- removed Raref1: 10k, Potentiometer_THT:Potentiometer_Piher_PT-15-V02_Vertical
- added J2: Conn_02x08_Odd_Even, Connector_PinSocket_2.54mm:PinSocket_2x08_P2.54mm_Vertical_SMD, F.Cu at (177.8, 58.4)
- Dprot1: footprint Diodes_SMD:D_SOD-123 -> Diode_SMD:D_SOD-123
- J1: value Conn_02x16_Counter_Clockwise -> Conn_02x18_Odd_Even; footprint One27:One27_male_32pin -> Connector_PinHeader_2.54mm:PinHeader_2x18_P2.54mm_Vertical_SMD
- Rref1: footprint Resistors_SMD:R_0805_HandSoldering -> Resistor_SMD:R_0805_2012Metric_Pad1.15x1.40mm_HandSolder
- moved Dprot1 55.4 mm to (193.0, 58.8)
- moved Rref1 55.1 mm to (198.1, 59.1)
- moved Jfpow1 43.8 mm to (139.8, 67.7), turned to 180 degrees
- moved Uout1 22.6 mm to (197.0, 92.2)
- moved J1 12.3 mm to (169.0, 95.3), turned to 0 degrees
- moved Uin1 3.58 mm to (141.0, 93.0)
Connections:
- Uin1 pad 16: Net-(J1-Pad16) -> Net-(J1-Pad33)
- Uin1 pad 17: Net-(J1-Pad15) -> Net-(J1-Pad31)
- Uin1 pad 18: Net-(J1-Pad14) -> Net-(J1-Pad29)
- Uin1 pad 19: Net-(J1-Pad13) -> Net-(J1-Pad27)
- Uin1 pad 2: Net-(J1-Pad8) -> Net-(J1-Pad17)
- Uin1 pad 20: Net-(J1-Pad12) -> Net-(J1-Pad25)
- Uin1 pad 21: Net-(J1-Pad11) -> Net-(J1-Pad23)
- Uin1 pad 22: Net-(J1-Pad10) -> Net-(J1-Pad21)
- Uin1 pad 23: Net-(J1-Pad9) -> Net-(J1-Pad19)
- Uin1 pad 3: Net-(J1-Pad7) -> Net-(J1-Pad15)
- Uin1 pad 4: Net-(J1-Pad6) -> Net-(J1-Pad13)
- Uin1 pad 5: Net-(J1-Pad5) -> Net-(J1-Pad11)
- Uin1 pad 6: Net-(J1-Pad4) -> Net-(J1-Pad9)
- Uin1 pad 7: Net-(J1-Pad3) -> Net-(J1-Pad7)
- Uin1 pad 8: Net-(J1-Pad2) -> Net-(J1-Pad5)
- Uin1 pad 9: Net-(J1-Pad1) -> Net-(J1-Pad3)
- Uout1 pad 16: Net-(J1-Pad32) -> Net-(J1-Pad4)
- Uout1 pad 17: Net-(J1-Pad31) -> Net-(J1-Pad6)
- Uout1 pad 18: Net-(J1-Pad30) -> Net-(J1-Pad8)
- Uout1 pad 19: Net-(J1-Pad29) -> Net-(J1-Pad10)
- Uout1 pad 2: Net-(J1-Pad24) -> Net-(J1-Pad20)
- Uout1 pad 20: Net-(J1-Pad28) -> Net-(J1-Pad12)
- Uout1 pad 21: Net-(J1-Pad27) -> Net-(J1-Pad14)
- Uout1 pad 22: Net-(J1-Pad26) -> Net-(J1-Pad16)
- Uout1 pad 23: Net-(J1-Pad25) -> Net-(J1-Pad18)
- Uout1 pad 3: Net-(J1-Pad23) -> Net-(J1-Pad22)
- Uout1 pad 4: Net-(J1-Pad22) -> Net-(J1-Pad24)
- Uout1 pad 5: Net-(J1-Pad21) -> Net-(J1-Pad26)
- Uout1 pad 6: Net-(J1-Pad20) -> Net-(J1-Pad28)
- Uout1 pad 7: Net-(J1-Pad19) -> Net-(J1-Pad30)
- Uout1 pad 8: Net-(J1-Pad18) -> Net-(J1-Pad32)
- Uout1 pad 9: Net-(J1-Pad17) -> Net-(J1-Pad34)
Routing:
- net /EN: track 83.0 -> 248.8 mm
- net /S6: track 56.6 -> 122.9 mm, vias 2 -> 0
- net /S7: track 53.1 -> 114.9 mm
- net /S3: track 52.2 -> 113.2 mm, vias 2 -> 0
- net /S2: track 45.2 -> 105.6 mm, vias 2 -> 0
- net Net-(Dprot1-Pad1): track 57.9 -> 112.3 mm
- net /S1: track 22.7 -> 64.4 mm
- net Net-(J1-Pad33): track 0.00 -> 38.5 mm
- net GND: track 184.5 -> 222.5 mm, vias 4 -> 5
- net Net-(J1-Pad34): track 0.00 -> 37.7 mm
- net /S0: track 22.2 -> 56.8 mm, vias 0 -> 2
- net Net-(J1-Pad1): track 24.0 -> 0.00 mm
- net Net-(J1-Pad2): track 22.6 -> 0.00 mm
- net Net-(J1-Pad25): track 12.9 -> 32.1 mm
- net Net-(J1-Pad9): track 14.2 -> 31.9 mm
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Other:
- board outline added: 86.4 x 76.1 mm

Commit message: Conversion perhaps works
Signed-off-by: byteofsoren <r00tr4t@gmail.com>
Routing:
- net /EN: track 248.8 -> 281.9 mm
- net GND: track 222.5 -> 205.4 mm
- net Net-(J1-Pad8): track 30.4 -> 46.1 mm
- net Net-(J1-Pad10): track 29.6 -> 44.9 mm
- net Net-(J1-Pad6): track 32.0 -> 47.3 mm
- net Net-(J1-Pad4): track 34.2 -> 48.6 mm
- net Net-(J1-Pad14): track 28.0 -> 41.7 mm
- net Net-(J1-Pad12): track 28.8 -> 41.9 mm
- net Net-(J1-Pad16): track 27.2 -> 37.9 mm
- net /S3: track 113.2 -> 103.1 mm
- net /S2: track 105.6 -> 96.3 mm
- net +5V: track 160.6 -> 152.8 mm
- net /S1: track 64.4 -> 57.0 mm, vias 0 -> 2
- net Net-(J1-Pad18): track 29.8 -> 36.0 mm
- net Net-(Dprot1-Pad1): track 112.3 -> 106.2 mm
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Other:
- board size 86.4 x 76.1 mm -> 91.4 x 78.7 mm
- net class Default: clearance 0.2 -> 0.5; via_drill 0.4 -> 0.6
- net class data added: clearance 0.5, trace_width 0.6, via_dia 1.5, via_drill 0.6
- rule trace_clearance: 0.2 -> 0.5
